File: esp32-c3-compact-dip-led.kicad_pcb (KiCad board)
At the start: 2 copper layers, 50 x 78 mm, 29 parts, among them J1 PJ-102A compatible 5.5/2.1mm, J2 USB-C POWER ONLY, J3 LED OUT, J4 M5STACK A105, Q1 RJP020N06T100, U1 ESP32-C3-WROOM-02-N4, U2 LMR36510FADDAR

Commit message: Use lower-cost 2A buck inductor
Parts:
- L1: value 22uH >=1.5A -> ZETC404020S-220MT-LF 22uH 2A Isat3.1A; footprint L_Vishay_IHLP-1616 -> Custom:ZETC404020S-220MT-LF
- moved L1 0.75 mm to (19.0, 55.2)
Routing:
- net REG_3V3: track 31.8 -> 35.5 mm, vias 3 -> 2
- net BUCK_SW: track 22.9 -> 23.5 mm
